Commit message: fixes and adding a second actuator

File: urdf/test.urdf (robot description, URDF)
Before this commit: robot dummy_robot, 2 links, 1 joints
Links:
- added link alt_link
Joints:
- added joint second: type continuous, parent base_link, child alt_link, origin xyz=0 0.3 0 rpy=0 0 0, axis 1 0 0
