Commit message: concrete exemple for a basic two Degrees-of-Freedom arm

File: urdf/sample.urdf (robot description, URDF)
Before this commit: robot dummy_robot, 3 links, 2 joints
Links:
- removed link alt_link
- added link middle_link; visual cylinder length=0.26 radius=0.04
- link base_link: geometry visual cylinder length=0.06 radius=0.04
- link end_link: geometry visual cylinder length=0.15 radius=0.04
Joints:
- removed joint first
- removed joint second
- added joint arm_joint_1: type revolute, parent base_link, child middle_link, origin xyz=0 0 0.06 rpy=0 0 0, axis 1 0 0, limit lower=-1.5708 upper=1.5708 effort=100 velocity=50
- added joint arm_joint_2: type revolute, parent middle_link, child end_link, origin xyz=0 0 0.26 rpy=0 0 0, axis 1 0 0, limit lower=-1.5708 upper=1.5708 effort=100 velocity=50

Commit message: change servo ids and joint limits

File: urdf/sample.urdf (robot description, URDF)
Before this commit: robot dummy_robot, 3 links, 2 joints
Joints:
- joint arm_joint_2: limit lower=-1.5708 upper=1.5708 effort=100 velocity=50 -> lower=-3.1415 upper=3.1415 effort=100 velocity=50

Commit message: Introduce support for joint limits as offered by ros_control

File: urdf/sample.urdf (robot description, URDF)
Before this commit: robot dummy_robot, 3 links, 2 joints
Joints:
- joint arm_joint_1: limit lower=-1.5708 upper=1.5708 effort=100 velocity=50 -> lower=-3.1415 upper=3.1415 effort=100 velocity=10
- joint arm_joint_2: limit lower=-3.1415 upper=3.1415 effort=100 velocity=50 -> lower=-3.1415 upper=3.1415 effort=100 velocity=5

Commit message: allow for a third joint in samble configs

File: urdf/sample.urdf (robot description, URDF)
Before this commit: robot dummy_robot, 3 links, 2 joints
Links:
- added link second_middle_link; visual cylinder length=0.26 radius=0.04
Joints:
- added joint arm_joint_3: type revolute, parent second_middle_link, child end_link, origin xyz=0 0 0.26 rpy=0 0 0, axis 1 0 0, limit lower=-3.1415 upper=3.1415 effort=100 velocity=10
- joint arm_joint_2: child end_link -> second_middle_link

Commit message: sample example update, working demo

File: urdf/sample.urdf (robot description, URDF)
Before this commit: robot dummy_robot, 4 links, 3 joints
Joints:
- joint arm_joint_1: limit lower=-3.1415 upper=3.1415 effort=100 velocity=10 -> lower=-10.1415 upper=10.1415 effort=100 velocity=10
- joint arm_joint_2: limit lower=-3.1415 upper=3.1415 effort=100 velocity=5 -> lower=-3.1415 upper=3.1415 effort=100 velocity=10
